File: Hardware/gatorBytes_Sensor_board.brd (EAGLE design)
At the start: 91.4 x 44.5 mm, 53 parts, among them U2 LIGHT_SENSORTEMT6000

Commit message: removing pth
Parts:
- removed D7: CLEAR, SparkFun-LED:LED-RGB-THRU
- removed U1: (no value), SparkFun-Sensors:TO-92-KIT
- added D1: XZM2CRKM2DGFBB45SCCB, SparkFun-LED:PLCC4SMDLED
- added U3: MCP9700TT, SparkFun-Sensors:SOT23-3
Connections:
- net 3.3V: now also D1.4, U3.1; no longer D7.2, U1.1
- net GND: now also U3.3; no longer U1.3
- net N$10: now also U3.2; no longer U1.2
- net N$11: now also D1.3; no longer D7.4
- net N$12: now also D1.1; no longer D7.1
- net N$13: now also D1.2; no longer D7.3
Routing:
- net N$13: track 4.53 -> 8.16 mm, vias 0 -> 2
- net N$10: track 7.24 -> 9.90 mm
- net 3.3V: track 277.8 -> 279.0 mm
- net GND: track 199.6 -> 200.6 mm, vias 0 -> 1
Changed lines of the file:
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@@
 <?xml version="1.0" encoding="utf-8"?>
 <!DOCTYPE eagle SYSTEM "eagle.dtd">
-<eagle version="8.7.0">
+<eagle version="9.1.0">
 <drawing>
 <settings>
@@
 <setting verticaltext="up"/>
 </settings>
-<grid distance="0.0125" unitdist="inch" unit="inch" style="lines" multiple="1" display="yes" altdistance="0.005" altunitdist="inch" altunit="inch"/>
+<grid distance="0.05" unitdist="inch" unit="inch" style="lines" multiple="1" display="yes" altdistance="0.005" altunitdist="inch" altunit="inch"/>
 <layers>
 <layer number="1" name="Top" color="4" fill="1" visible="yes" active="yes"/>
@@
 <param name="checkStop" value="0"/>
 <param name="checkValues" value="0"/>
+<param name="checkNames" value="1"/>
+<param name="checkWireStubs" value="1"/>
+<param name="checkPolygonWidth" value="0"/>
 <param name="useDiameter" value="13"/>
 <param name="maxErrors" value="50"/>
@@
 </autorouter>
 <elements>
-<element name="D7" library="SparkFun-LED" package="LED-RGB-THRU" value="CLEAR" x="45.72" y="22.225" rot="R180">
-<attribute name="PROD_ID" value="DIO-08418" x="45.72" y="22.225" size="1.778" layer="27" rot="R180" display="off"/>
-</element>
 <element name="FRAME1" library="SparkFun-Aesthetics" package="CREATIVE_COMMONS" value="FRAME-LETTER" x="22.225" y="-9.525"/>
 <element name="R10" library="SparkFun-Resistors" package="0603" value="100" x="45.72" y="17.78">
@@
 <element name="U$25" library="TAB" package="GATOR_MINI" value="GATOR_MINI" x="69.85" y="8.89"/>
 <element name="U$26" library="TAB" package="GATOR_MINI" value="GATOR_MINI" x="81.28" y="8.89"/>
-<element name="U1" library="SparkFun-Sensors" package="TO-92-KIT" value="" x="15.875" y="20.32">
-<attribute name="PROD_ID" value="IC-09880" x="15.875" y="20.32" size="1.778" layer="27" display="off"/>
-<attribute name="SF_ID" value="SEN-10988" x="15.875" y="20.32" size="1.778" layer="27" display="off"/>
-</element>
 <element name="U2" library="SparkFun-Sensors" package="TEMT6000" value="LIGHT_SENSORTEMT6000" x="75.565" y="21.59" rot="R180">
 <attribute name="PROD_ID" value="COMP-08569" x="75.565" y="21.59" size="1.778" layer="27" rot="R180" display="off"/>
@@
 <element name="U$5" library="SparkFun-Aesthetics" package="SFE_LOGO_NAME_FLAME_.1" value="" x="69.85" y="38.1"/>
 <element name="U$33" library="SparkFun-Aesthetics" package="ORDERING_INSTRUCTIONS" value="" x="-3.81" y="-12.065"/>
+<element name="U3" library="SparkFun-Sensors" package="SOT23-3" value="MCP9700TT" x="15.875" y="20.955">
+<attribute name="PROD_ID" value="IC-08917" x="15.875" y="20.955" size="1.778" layer="27" display="off"/>
+</element>
+<element name="D1" library="SparkFun-LED" package="PLCC4SMDLED" value="XZM2CRKM2DGFBB45SCCB" x="45.72" y="22.225">
+<attribute name="PROD_ID" value="DIO-13722" x="45.72" y="22.225" size="1.778" layer="27" display="off"/>
+</element>
 </elements>
 <signals>
 <signal name="3.3V">
-<contactref element="D7" pad="2"/>
 <contactref element="U$12" pad="P1"/>
 <contactref element="U$11" pad="P1"/>
-<contactref element="U1" pad="1"/>
 <contactref element="U2" pad="COLLECTOR"/>
 <contactref element="U$26" pad="P1"/>
-<wire x1="45.085" y1="22.225" x2="45.3644" y2="22.5044" width="0.4064" layer="1"/>
-<wire x1="45.3644" y1="22.5044" x2="45.3644" y2="23.270325" width="0.4064" layer="1"/>
-<wire x1="45.3644" y1="23.270325" x2="45.72" y2="23.625925" width="0.4064" layer="1"/>
-<wire x1="45.72" y1="23.625925" x2="45.72" y2="27.305" width="0.4064" layer="1"/>
 <wire x1="45.72" y1="27.305" x2="45.72" y2="33.274" width="0.4064" layer="1"/>
 <wire x1="73.705" y1="21.58" x2="73.705" y2="23.159" width="0.4064" layer="1"/>
@@
 <wire x1="80.645" y1="22.479" x2="78.994" y2="24.13" width="0.4064" layer="1"/>
 <wire x1="78.994" y1="24.13" x2="74.676" y2="24.13" width="0.4064" layer="1"/>
-<wire x1="14.605" y1="20.32" x2="14.605" y2="14.859" width="0.4064" layer="1"/>
-<wire x1="14.605" y1="14.859" x2="15.748" y2="13.716" width="0.4064" layer="1"/>
-<wire x1="15.748" y1="13.716" x2="21.59" y2="13.716" width="0.4064" layer="1"/>
+<wire x1="21.59" y1="13.716" x2="15.748" y2="13.716" width="0.4064" layer="1"/>
 <wire x1="21.59" y1="13.716" x2="21.59" y2="18.415" width="0.4064" layer="16"/>
 <wire x1="21.59" y1="18.415" x2="24.13" y2="20.955" width="0.4064" layer="16"/>
@@
 <wire x1="82.55" y1="20.955" x2="81.28" y2="19.685" width="0.4064" layer="16"/>
 <wire x1="81.28" y1="19.685" x2="81.28" y2="13.716" width="0.4064" layer="16"/>
+<contactref element="U3" pad="1"/>
+<wire x1="15.748" y1="13.716" x2="14.925" y2="14.539" width="0.4064" layer="1"/>
+<wire x1="14.925" y1="14.539" x2="14.925" y2="19.955" width="0.4064" layer="1"/>
+<contactref element="D1" pad="4"/>
+<wire x1="44.32" y1="21.5" x2="45.376" y2="21.5" width="0.4064" layer="1"/>
+<wire x1="45.376" y1="21.5" x2="45.72" y2="21.844" width="0.4064" layer="1"/>
+<wire x1="45.72" y1="21.844" x2="45.72" y2="27.305" width="0.4064" layer="1"/>
 </signal>
 <signal name="GND">
 <contactref element="U$22" pad="P1"/>
-<contactref element="U1" pad="3"/>
 <contactref element="R11" pad="1"/>
 <contactref element="U$25" pad="P1"/>
-<wire x1="17.145" y1="20.32" x2="17.145" y2="16.129" width="0.4064" layer="16"/>
-<wire x1="14.732" y1="13.716" x2="17.145" y2="16.129" width="0.4064" layer="16"/>
 <wire x1="10.16" y1="13.716" x2="12.954" y2="13.716" width="0.4064" layer="1"/>
 <wire x1="12.954" y1="13.716" x2="15.875" y2="10.795" width="0.4064" layer="1"/>
 <wire x1="15.875" y1="4.445" x2="18.415" y2="1.905" width="0.4064" layer="1"/>
 <wire x1="15.875" y1="10.795" x2="15.875" y2="4.445" width="0.4064" layer="1"/>
-<wire x1="10.16" y1="13.716" x2="14.732" y2="13.716" width="0.4064" layer="16"/>
 <wire x1="10.16" y1="13.716" x2="12.954" y2="13.716" width="0.4064" layer="16"/>
 <wire x1="12.954" y1="13.716" x2="15.875" y2="10.795" width="0.4064" layer="16"/>
@@
 <wire x1="71.4375" y1="19.05" x2="69.85" y2="17.4625" width="0.4064" layer="1"/>
 <wire x1="69.85" y1="17.4625" x2="69.85" y2="13.716" width="0.4064" layer="1"/>
+<contactref element="U3" pad="3"/>
+<wire x1="10.16" y1="13.716" x2="14.351" y2="13.716" width="0.4064" layer="16"/>
+<wire x1="14.351" y1="13.716" x2="15.875" y2="15.24" width="0.4064" layer="16"/>
+<wire x1="15.875" y1="15.24" x2="15.875" y2="17.145" width="0.4064" layer="16"/>
+<via x="15.875" y="17.145" extent="1-16" drill="0.381"/>
+<wire x1="15.875" y1="17.145" x2="15.875" y2="22.055" width="0.4064" layer="1"/>
 </signal>
 <signal name="N$11">
-<contactref element="D7" pad="4"/>
 <contactref element="R9" pad="2"/>
-<wire x1="47.625" y1="22.225" x2="48.475" y2="21.375" width="0.4064" layer="1"/>
-<wire x1="48.475" y1="21.375" x2="50.165" y2="21.375" width="0.4064" layer="1"/>
+<contactref element="D1" pad="3"/>
+<wire x1="50.165" y1="21.375" x2="50.04" y2="21.5" width="0.4064" layer="1"/>
+<wire x1="50.04" y1="21.5" x2="47.12" y2="21.5" width="0.4064" layer="1"/>
 </signal>
 <signal name="N$12">
-<contactref element="D7" pad="1"/>
 <contactref element="R8" pad="2"/>
-<wire x1="41.91" y1="23.075" x2="42.965" y2="23.075" width="0.4064" layer="1"/>
-<wire x1="42.965" y1="23.075" x2="43.815" y2="22.225" width="0.4064" layer="1"/>
+<wire x1="42.965" y1="23.075" x2="41.91" y2="23.075" width="0.4064" layer="1"/>
+<contactref element="D1" pad="1"/>
+<wire x1="44.32" y1="22.95" x2="43.09" y2="22.95" width="0.4064" layer="1"/>
+<wire x1="43.09" y1="22.95" x2="42.965" y2="23.075" width="0.4064" layer="1"/>
 </signal>
 <signal name="N$13">
-<contactref element="D7" pad="3"/>
 <contactref element="R10" pad="2"/>
-<wire x1="46.355" y1="22.225" x2="46.57" y2="22.01" width="0.4064" layer="1"/>
-<wire x1="46.57" y1="22.01" x2="46.57" y2="17.78" width="0.4064" layer="1"/>
+<contactref element="D1" pad="2"/>
+<wire x1="47.12" y1="22.95" x2="48.424" y2="22.95" width="0.4064" layer="1"/>
+<wire x1="48.424" y1="22.95" x2="48.514" y2="22.86" width="0.4064" layer="1"/>
+<via x="48.514" y="22.86" extent="1-16" drill="0.381"/>
+<wire x1="48.514" y1="22.86" x2="48.514" y2="19.05" width="0.4064" layer="16"/>
+<via x="48.514" y="19.05" extent="1-16" drill="0.381"/>
+<wire x1="48.514" y1="19.05" x2="48.514" y2="18.288" width="0.4064" layer="1"/>
+<wire x1="48.514" y1="18.288" x2="48.006" y2="17.78" width="0.4064" layer="1"/>
+<wire x1="48.006" y1="17.78" x2="46.57" y2="17.78" width="0.4064" layer="1"/>
 </signal>
 <signal name="N$14">
@@
 </signal>
 <signal name="N$10">
-<contactref element="U1" pad="2"/>
 <contactref element="U$23" pad="P1"/>
-<wire x1="15.875" y1="29.464" x2="15.875" y2="22.225" width="0.4064" layer="1"/>
+<contactref element="U3" pad="2"/>
+<wire x1="16.825" y1="19.955" x2="16.825" y2="23.4975" width="0.4064" layer="1"/>
+<wire x1="16.825" y1="23.4975" x2="15.875" y2="24.4475" width="0.4064" layer="1"/>
+<wire x1="15.875" y1="24.4475" x2="15.875" y2="29.464" width="0.4064" layer="1"/>
 </signal>
 <signal name="N$18">
@@
 </signal>
 </signals>
+<mfgpreviewcolors>
+<mfgpreviewcolor name="soldermaskcolor" color="0xC8008000"/>
+<mfgpreviewcolor name="silkscreencolor" color="0xFFFEFEFE"/>
+<mfgpreviewcolor name="backgroundcolor" color="0xFF282828"/>
+<mfgpreviewcolor name="coppercolor" color="0xFFFFBF00"/>
+<mfgpreviewcolor name="substratecolor" color="0xFF786E46"/>
+</mfgpreviewcolors>
 <errors>
 </errors>

Commit message: adding new tabs
Parts:
- added U$35: GATOR_MINI, TAB:GATOR_MINI
- added U$36, U$37: (no value), 001:3#3V1
- added U$38, U$39: (no value), 001:GND0
- added U$40: (no value), buzzard_labels (1):RGB0
- added U$41: (no value), gator#PNG (6):GATOR#PNG
- D1: device SparkFun-LED:PLCC4SMDLED -> SparkFun-LED:LED-TRICOLOR-SMD
- U$10, U$14, U$15, U$23, U$24: value GATOR_MINI -> GATOR; device TAB:GATOR_MINI -> SparkFun-Connectors:GATOR
- U$19: value (none) -> GATOR_MINI; device 002:TRI#COLOR5 -> TAB:GATOR_MINI
- U$30: device 003:GATORBYTES6 -> buzzard_labels (4):GATOR#STARTER0
- moved U$5 62.1 mm to (19.4, 1.78)
- moved U$27 44.6 mm to (44.7, 46.4)
- moved U$30 44.0 mm to (33.0, 3.81)
- moved U$16 43.2 mm to (10.3, 45.7)
- moved U$17 43.2 mm to (6.22, 48.3)
- moved U$20 43.2 mm to (71.1, 48.3)
- moved U$21 43.2 mm to (70.0, 45.8)
- moved U$19 28.9 mm to (6.99, 0.64)
- moved U$10 13.8 mm to (37.5, 19.6)
- moved U$14 13.8 mm to (54.0, 19.6)
- moved U$15 13.8 mm to (45.7, 19.6)
- moved R10 8.89 mm to (45.7, 26.7)
- moved U$8 8.89 mm to (41.7, 24.3)
- moved U$18 8.89 mm to (34.5, 24.1)
- moved U$4 8.89 mm to (50.5, 24.1)
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Connections:
- net 3.3V: now also D1.A, U$19.P1; no longer D1.4
- net GND: now also U$35.P1
- net N$10: now also U$23.P$1, U$23.P$2; no longer U$23.P1
- net N$11: now also D1.B; no longer D1.3
- net N$12: now also D1.R; no longer D1.1
- net N$13: now also D1.G; no longer D1.2
- net N$14: now also U$10.P$1, U$10.P$2; no longer U$10.P1
- net N$15: now also U$14.P$1, U$14.P$2; no longer U$14.P1
- net N$16: now also U$15.P$1, U$15.P$2; no longer U$15.P1
- net N$18: now also U$24.P$1, U$24.P$2; no longer U$24.P1
Routing:
- net 3.3V: track 279.0 -> 428.0 mm
- net GND: track 200.6 -> 211.7 mm
- net N$18: track 17.1 -> 6.76 mm
- net N$10: track 9.90 -> 16.3 mm
- net N$14: track 12.7 -> 11.5 mm
- net N$13: track 8.16 -> 7.07 mm
- net N$15: track 15.4 -> 14.7 mm
Other:
- board size 91.4 x 44.5 mm -> 91.4 x 49.5 mm
- board text added: "v02"
- board text removed: "v01"

Commit message: post design review changes
Routing:
- net 3.3V: track 428.0 -> 471.5 mm
- net N$18: track 6.76 -> 25.0 mm
Other:
- outline, holes or cut-outs redrawn

Commit message: post checklist chanegs
Parts:
- D1: device SparkFun-LED:LED-TRICOLOR-SMD -> SparkFun-LED:PLCC4SMDLED
- U$1: device 001:3#3V1 -> 001:GND0
- U$11, U$12, U$19, U$22, U$25, U$26, U$35: value GATOR_MINI -> TAB_GATOR_MINI; device TAB:GATOR_MINI -> SparkFun-Connectors:TAB_GATOR_MINI
- U$23: value GATOR -> TAB_GATOR_MINI; device SparkFun-Connectors:GATOR -> SparkFun-Connectors:TAB_GATOR_MINI
- moved U$23 10.2 mm to (15.9, 41.9)
- moved U$27 1.27 mm to (44.7, 47.6)
- moved U$40 1.27 mm to (39.6, 47.6)
- moved U$1 0.13 mm to (42.7, 33.7)
- turned D1 to 0 degrees
Connections:
- net 3.3V: no longer D1.A, U$12.P1
- net GND: now also D1.4, U$12.P1
- net N$10: now also U$23.P1; no longer U$23.P$1, U$23.P$2
- net N$11: now also D1.3; no longer D1.B
- net N$12: now also D1.1; no longer D1.R
- net N$13: now also D1.2; no longer D1.G
Routing:
- net GND: track 211.7 -> 281.8 mm
- net 3.3V: track 471.5 -> 442.1 mm
- net N$15: track 14.7 -> 23.0 mm
- net N$18: track 25.0 -> 30.8 mm
- net N$14: track 11.5 -> 17.4 mm
- net N$16: track 7.72 -> 13.6 mm
- net N$10: track 16.3 -> 15.0 mm
Other:
- board text added: "v10"
- board text removed: "v02"

Commit message: post qc checklist
Parts:
- added LOGO7: REVISION, SparkFun-Aesthetics:REVISION
- moved U$8 0.13 mm to (41.7, 24.1)
Other:
- board text added: "A. England"
Changed lines of the file:
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@@
 <hole x="5.08" y="26.416" drill="0.381"/>
 <hole x="5.08" y="25.4" drill="0.381"/>
-<hole x="26.67" y="27.813" drill="0.381"/>
-<hole x="26.67" y="24.257" drill="0.381"/>
+<hole x="26.67" y="26.543" drill="0.381"/>
+<hole x="26.67" y="25.527" drill="0.381"/>
 <hole x="33.02" y="26.543" drill="0.381"/>
 <hole x="33.02" y="25.527" drill="0.381"/>
@@
 <hole x="15.367" y="10.541" drill="0.381"/>
 <hole x="16.383" y="10.541" drill="0.381"/>
-<hole x="43.942" y="44.069" drill="0.381"/>
-<hole x="47.498" y="44.069" drill="0.381"/>
+<hole x="45.212" y="44.069" drill="0.381"/>
+<hole x="46.228" y="44.069" drill="0.381"/>
 <hole x="58.42" y="25.527" drill="0.381"/>
 <hole x="58.42" y="26.543" drill="0.381"/>
@@
 <hole x="75.057" y="42.799" drill="0.381"/>
 <hole x="76.073" y="42.799" drill="0.381"/>
-<hole x="86.487" y="27.813" drill="0.381"/>
-<hole x="86.487" y="24.257" drill="0.381"/>
+<hole x="86.487" y="26.543" drill="0.381"/>
+<hole x="86.487" y="25.527" drill="0.381"/>
 <wire x1="76.454" y1="10.795" x2="76.454" y2="9.525" width="0.2032" layer="20"/>
 <wire x1="76.454" y1="9.525" x2="86.36" y2="9.525" width="0.2032" layer="20"/>
@@
 <wire x1="85.09" y1="42.545" x2="76.5175" y2="42.545" width="0.254" layer="51"/>
 <wire x1="76.5175" y1="42.545" x2="76.5175" y2="43.815" width="0.254" layer="51"/>
-<text x="4.826" y="26.2255" size="0.8128" layer="51" font="vector" ratio="15" rot="R90">route out</text>
-<text x="12.5095" y="43.561" size="0.8128" layer="51" font="vector" ratio="15" rot="R180">route out</text>
-<text x="22.6695" y="43.561" size="0.8128" layer="51" font="vector" ratio="15" rot="R180">route out</text>
-<text x="26.924" y="33.147" size="0.8128" layer="51" font="vector" ratio="15" rot="R270">route out</text>
-<text x="26.924" y="23.622" size="0.8128" layer="51" font="vector" ratio="15" rot="R270">route out</text>
-<text x="19.2405" y="9.779" size="0.8128" layer="51" font="vector" ratio="15">route out</text>
-<text x="8.4455" y="9.779" size="0.8128" layer="51" font="vector" ratio="15">route out</text>
-<text x="4.826" y="14.478" size="0.8128" layer="51" font="vector" ratio="15" rot="R90">route out</text>
-<text x="32.766" y="16.7005" size="0.8128" layer="51" font="vector" ratio="15" rot="R90">route out</text>
-<text x="37.338" y="7.874" size="0.8128" layer="51" font="vector" ratio="15">route out</text>
-<text x="48.4505" y="7.874" size="0.8128" layer="51" font="vector" ratio="15">route out</text>
-<text x="59.436" y="17.653" size="0.8128" layer="51" font="vector" ratio="15" rot="R90">route out</text>
-<text x="59.436" y="29.4005" size="0.8128" layer="51" font="vector" ratio="15" rot="R90">route out</text>
-<text x="48.768" y="44.069" size="0.8128" layer="51" font="vector" ratio="15">route out</text>
-<text x="37.338" y="44.069" size="0.8128" layer="51" font="vector" ratio="15">route out</text>
-<text x="37.338" y="44.069" size="0.8128" layer="51" font="vector" ratio="15">route out</text>
-<text x="32.766" y="31.623" size="0.8128" layer="51" font="vector" ratio="15" rot="R90">route out</text>
-<text x="67.5005" y="42.799" size="0.8128" layer="51" font="vector" ratio="15">route out</text>
-<text x="77.6605" y="42.799" size="0.8128" layer="51" font="vector" ratio="15">route out</text>
-<text x="64.516" y="26.2255" size="0.8128" layer="51" font="vector" ratio="15" rot="R90">route out</text>
-<text x="87.376" y="28.7655" size="0.8128" layer="51" font="vector" ratio="15" rot="R90">route out</text>
-<text x="87.376" y="16.383" size="0.8128" layer="51" font="vector" ratio="15" rot="R90">route out</text>
-<text x="64.516" y="16.7005" size="0.8128" layer="51" font="vector" ratio="15" rot="R90">route out</text>
-<text x="72.1995" y="10.541" size="0.8128" layer="51" font="vector" ratio="15" rot="R180">route out</text>
-<text x="83.312" y="10.541" size="0.8128" layer="51" font="vector" ratio="15" rot="R180">route out</text>
+<text x="4.826" y="28.7655" size="0.8128" layer="20" font="vector" ratio="15" rot="R90">route out</text>
+<text x="12.5095" y="43.561" size="0.8128" layer="20" font="vector" ratio="15" rot="R180">route out</text>
+<text x="22.6695" y="43.561" size="0.8128" layer="20" font="vector" ratio="15" rot="R180">route out</text>
+<text x="26.924" y="33.147" size="0.8128" layer="20" font="vector" ratio="15" rot="R270">route out</text>
+<text x="26.924" y="23.622" size="0.8128" layer="20" font="vector" ratio="15" rot="R270">route out</text>
+<text x="19.2405" y="9.779" size="0.8128" layer="20" font="vector" ratio="15">route out</text>
+<text x="8.4455" y="9.779" size="0.8128" layer="20" font="vector" ratio="15">route out</text>
+<text x="4.826" y="14.478" size="0.8128" layer="20" font="vector" ratio="15" rot="R90">route out</text>
+<text x="32.766" y="16.7005" size="0.8128" layer="20" font="vector" ratio="15" rot="R90">route out</text>
+<text x="37.338" y="7.874" size="0.8128" layer="20" font="vector" ratio="15">route out</text>
+<text x="48.4505" y="7.874" size="0.8128" layer="20" font="vector" ratio="15">route out</text>
+<text x="59.436" y="17.653" size="0.8128" layer="20" font="vector" ratio="15" rot="R90">route out</text>
+<text x="59.436" y="29.4005" size="0.8128" layer="20" font="vector" ratio="15" rot="R90">route out</text>
+<text x="48.768" y="44.069" size="0.8128" layer="20" font="vector" ratio="15">route out</text>
+<text x="36.068" y="44.069" size="0.8128" layer="20" font="vector" ratio="15">route out</text>
+<text x="32.766" y="31.623" size="0.8128" layer="20" font="vector" ratio="15" rot="R90">route out</text>
+<text x="67.5005" y="42.799" size="0.8128" layer="20" font="vector" ratio="15">route out</text>
+<text x="77.6605" y="42.799" size="0.8128" layer="20" font="vector" ratio="15">route out</text>
+<text x="64.516" y="28.7655" size="0.8128" layer="20" font="vector" ratio="15" rot="R90">route out</text>
+<text x="87.376" y="28.7655" size="0.8128" layer="20" font="vector" ratio="15" rot="R90">route out</text>
+<text x="87.376" y="16.383" size="0.8128" layer="20" font="vector" ratio="15" rot="R90">route out</text>
+<text x="64.516" y="16.7005" size="0.8128" layer="20" font="vector" ratio="15" rot="R90">route out</text>
+<text x="72.1995" y="10.541" size="0.8128" layer="20" font="vector" ratio="15" rot="R180">route out</text>
+<text x="83.312" y="10.541" size="0.8128" layer="20" font="vector" ratio="15" rot="R180">route out</text>
 <text x="4.15925" y="-31.1785" size="2.54" layer="51">Solder Mask: Black Gloss</text>
 <dimension x1="1.27" y1="49.53" x2="1.27" y2="0" x3="-2.54" y3="24.765" textsize="1.778" layer="47" unit="inch"/>
 <dimension x1="0" y1="48.26" x2="91.44" y2="48.26" x3="45.72" y3="52.07" textsize="1.778" layer="47" unit="inch"/>
+<text x="48.26" y="-11.684" size="1.778" layer="51" font="vector" ratio="15">A. England</text>
 </plain>
 <attributes>
@@
 <element name="U$6" library="001" package="GND0" value="" x="7.112" y="20.955"/>
 <element name="U$7" library="001" package="GND0" value="" x="67.437" y="20.955"/>
-<element name="U$8" library="001" package="GREEN9" value="" x="41.656" y="24.257"/>
+<element name="U$8" library="001" package="GREEN9" value="" x="41.656" y="24.13"/>
 <element name="U$9" library="001" package="LIGHT4" value="" x="71.882" y="27.305"/>
 <element name="U$13" library="001" package="TEMP3" value="" x="12.065" y="27.305"/>
@@
 <element name="U$30" library="buzzard_labels (4)" package="GATOR#STARTER0" value="" x="33.02" y="3.81"/>
 <element name="U$1" library="001" package="GND0" value="" x="42.672" y="33.655"/>
+<element name="LOGO7" library="SparkFun-Aesthetics" package="REVISION" value="REVISION" x="33.782" y="-11.684"/>
 </elements>
 <signals>
