File: Hardware/gatorBytes_Sensor_board.brd (EAGLE design)
At the start: 91.4 x 49.5 mm, 61 parts, among them U2 LIGHT_SENSORTEMT6000, U3 MCP9700TT

Commit message: silk update
Parts:
- U$23: value TAB_GATOR_MINI -> GATOR; device SparkFun-Connectors:TAB_GATOR_MINI -> SparkFun-Connectors:GATOR
- U$34: device 003:TRI#COLOR_LED1 -> buzzard_labels (1):RGB_LED0
- moved U$23 10.2 mm to (15.9, 31.8)
- moved U$34 1.80 mm to (49.7, 31.7)
Connections:
- net N$10: now also U$23.P$1, U$23.P$2; no longer U$23.P1
Routing:
- net N$10: track 15.0 -> 18.9 mm
Changed lines of the file:
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@@
 <element name="U$15" library="SparkFun-Connectors" package="GATOR" value="GATOR" x="45.72" y="19.558"/>
 <element name="U$22" library="SparkFun-Connectors" package="TAB_GATOR_MINI" value="TAB_GATOR_MINI" x="10.16" y="11.43"/>
-<element name="U$23" library="SparkFun-Connectors" package="TAB_GATOR_MINI" value="TAB_GATOR_MINI" x="15.875" y="41.91" rot="R180"/>
+<element name="U$23" library="SparkFun-Connectors" package="GATOR" value="GATOR" x="15.875" y="31.75" rot="R180"/>
 <element name="U$24" library="SparkFun-Connectors" package="GATOR" value="GATOR" x="75.565" y="31.75" rot="R180"/>
 <element name="U$25" library="SparkFun-Connectors" package="TAB_GATOR_MINI" value="TAB_GATOR_MINI" x="69.85" y="11.43"/>
@@
 <element name="U$31" library="003" package="LIGHT_SENSOR0" value="" x="80.645" y="27.305" rot="MR0"/>
 <element name="U$32" library="003" package="TEMP_SENSOR3" value="" x="25.0825" y="26.9875" rot="MR0"/>
-<element name="U$34" library="003" package="TRI#COLOR_LED1" value="" x="51.435" y="31.4325" rot="MR0"/>
+<element name="U$34" library="buzzard_labels (1)" package="RGB_LED0" value="" x="49.657" y="31.6865" rot="MR0"/>
 <element name="U$5" library="SparkFun-Aesthetics" package="SFE_LOGO_NAME_FLAME_.1" value="" x="19.431" y="1.778"/>
 <element name="U$33" library="SparkFun-Aesthetics" package="ORDERING_INSTRUCTIONS" value="" x="-3.81" y="-12.065"/>
@@
 </signal>
 <signal name="N$10">
-<contactref element="U$23" pad="P1"/>
+<contactref element="U$23" pad="P$1"/>
 <contactref element="U3" pad="2"/>
-<wire x1="15.875" y1="29.845" x2="15.875" y2="37.084" width="0.4064" layer="1"/>
-<wire x1="16.825" y1="22.495" x2="16.825" y2="28.895" width="0.4064" layer="1"/>
-<wire x1="16.825" y1="28.895" x2="15.875" y2="29.845" width="0.4064" layer="1"/>
+<wire x1="15.875" y1="29.845" x2="15.875" y2="33.02" width="0.4064" layer="1"/>
+<contactref element="U$23" pad="P$2"/>
+<wire x1="15.875" y1="33.02" x2="15.875" y2="37.846" width="0.4064" layer="1"/>
+<wire x1="15.875" y1="32.004" x2="15.875" y2="27.305" width="0.4064" layer="1"/>
+<wire x1="16.825" y1="26.355" x2="16.825" y2="22.495" width="0.4064" layer="1"/>
+<wire x1="15.875" y1="27.305" x2="16.825" y2="26.355" width="0.4064" layer="1"/>
+<wire x1="15.875" y1="32.004" x2="15.875" y2="33.02" width="0.4064" layer="1"/>
 </signal>
 <signal name="N$18">
