File: Production/14062-gatorBytes_Sensor_board-Panel.brd (EAGLE design)
At the start: 111.5 x 119.6 mm, 119 parts, among them U1 LIGHT_SENSORTEMT6000, U2 LIGHT_SENSORTEMT6000, U3 MCP9700TT, U4 MCP9700TT

Commit message: panel
Parts:
- removed E$2: (no value), SparkFun-Aesthetics:FIDUCIAL-1X2
- added D3, D4, D5, D6: XZM2CRKM2DGFBB45SCCB, SparkFun-LED:PLCC4SMDLED
- added E$4: (no value), SparkFun-Retired:FIDUCIAL-1.5X3
- added E$5, E$6: (no value), SparkFun-Aesthetics:FIDUCIAL-1X2
- added FD10, FD11, FD12, FD13, FD14, FD15, FD16, FD17, FD18, FD19, FD20, FD21, FD22, FD23, FD24, FD9: FIDUCIALUFIDUCIAL, SparkFun-Aesthetics:FIDUCIAL-MICRO
- added LOGO13, LOGO16, LOGO18, LOGO19, LOGO22, LOGO24, LOGO25, LOGO28, LOGO30, LOGO31, LOGO34, LOGO36: SFE_LOGO_FLAME.1_INCH, SparkFun-Aesthetics:SFE_LOGO_FLAME_.1
- added LOGO14, LOGO15, LOGO17, LOGO20, LOGO21, LOGO23, LOGO26, LOGO27, LOGO29, LOGO32, LOGO33, LOGO35: OSHW-LOGOS, SparkFun-Aesthetics:OSHW-LOGO-S
- added R12, R13, R16, R17, R20, R21, R24, R5: 100, SparkFun-Resistors:0603
- added R14, R18, R22, R6: 10k, SparkFun-Resistors:0603
- added R15, R19, R23, R7: 200, SparkFun-Resistors:0603
- added U$100, U$141, U$182, U$223: (no value), 001:TEMP3
- added U$101, U$142, U$183, U$224: (no value), 001:RED8
- added U$102, U$143, U$184, U$225: (no value), 002:TEMPERATURE3
- added U$103, U$105, U$144, U$146, U$185, U$187, U$226, U$228: (no value), 002:SENSOR2
- added U$104, U$145, U$186, U$227: (no value), 002:LIGHT4
- added U$106, U$147, U$188, U$229: (no value), 002:LED5
- added U$107, U$108, U$109, U$121, U$148, U$149, U$150, U$162, U$189, U$190, U$191, U$203, U$230, U$231, U$232, U$244: (no value), gator#PNG (6):GATOR#PNG
- added U$110, U$151, U$192, U$233: (no value), 003:LIGHT_SENSOR0
- added U$111, U$152, U$193, U$234: (no value), 003:TEMP_SENSOR3
- added U$112, U$153, U$194, U$235: (no value), 003:TRI#COLOR_LED1
- added U$113, U$154, U$195, U$236: (no value), SparkFun-Aesthetics:SFE_LOGO_NAME_FLAME_.1
- added U$114, U$115, U$125, U$126, U$129, U$130, U$132, U$133, U$155, U$156, U$166, U$167, U$170, U$171, U$173, U$174, U$196, U$197, U$207, U$208, U$211, U$212, U$214, U$215, U$237, U$238, U$84, U$85, U$88, U$89, U$91, U$92: TAB_GATOR_MINI, SparkFun-Connectors:TAB_GATOR_MINI
- added U$116, U$117, U$134, U$135, U$157, U$158, U$175, U$176, U$198, U$199, U$216, U$217, U$239, U$240, U$93, U$94: (no value), 001:3#3V1
- added U$118, U$119, U$123, U$137, U$138, U$159, U$160, U$164, U$178, U$179, U$200, U$201, U$205, U$219, U$220, U$241, U$242, U$246, U$96, U$97: (no value), 001:GND0
- added U$120, U$161, U$202, U$243: (no value), buzzard_labels (1):RGB0
- added U$122, U$163, U$204, U$245: (no value), buzzard_labels (4):GATOR#STARTER0
- added U$124, U$127, U$128, U$131, U$165, U$168, U$169, U$172, U$206, U$209, U$210, U$213, U$83, U$86, U$87, U$90: GATOR, SparkFun-Connectors:GATOR
- added U$136, U$177, U$218, U$95: (no value), 001:BLUE10
- added U$139, U$180, U$221, U$98: (no value), 001:GREEN9
- added U$140, U$181, U$222, U$99: (no value), 001:LIGHT4
- added U10, U12, U6, U8: MCP9700TT, SparkFun-Sensors:SOT23-3
- added U11, U5, U7, U9: LIGHT_SENSORTEMT6000, SparkFun-Sensors:TEMT6000
- moved E$1 212.4 mm to (93.6, 295.5), turned to 90 degrees
- moved E$3 18.7 mm to (-4.19, 13.0), turned to 180 degrees
Connections:
- new net 3.3V2: U$114.P1, U$84.P1, U$92.P1, U5.COLLECTOR, U6.1
- new net 3.3V3: U$125.P1, U$133.P1, U$155.P1, U7.COLLECTOR, U8.1
- new net 3.3V4: U$166.P1, U$174.P1, U$196.P1, U10.1, U9.COLLECTOR
- new net 3.3V5: U$207.P1, U$215.P1, U$237.P1, U11.COLLECTOR, U12.1
- new net GND2: D3.4, R6.1, U$115.P1, U$85.P1, U$88.P1, U$91.P1, U6.3
- new net GND3: D4.4, R14.1, U$126.P1, U$129.P1, U$132.P1, U$156.P1, U8.3
- new net GND4: D5.4, R18.1, U$167.P1, U$170.P1, U$173.P1, U$197.P1, U10.3
- new net GND5: D6.4, R22.1, U$208.P1, U$211.P1, U$214.P1, U$238.P1, U12.3
- new net N$17: D3.1, R7.2
- new net N$19: D3.2, R5.2
- new net N$20: R7.1, U$83.P$1, U$83.P$2
- new net N$21: R12.1, U$86.P$1, U$86.P$2
- new net N$22: R5.1, U$87.P$1, U$87.P$2
- new net N$23: U$89.P1, U6.2
- new net N$24: R6.2, U$90.P$1, U$90.P$2, U5.EMITTER
- new net N$25: D4.3, R16.2
- new net N$26: D4.1, R15.2
- new net N$27: D4.2, R13.2
- new net N$28: R15.1, U$124.P$1, U$124.P$2
- new net N$29: R16.1, U$127.P$1, U$127.P$2
- new net N$30: R13.1, U$128.P$1, U$128.P$2
- new net N$31: U$130.P1, U8.2
- new net N$32: R14.2, U$131.P$1, U$131.P$2, U7.EMITTER
- new net N$33: D5.3, R20.2
- new net N$34: D5.1, R19.2
- new net N$35: D5.2, R17.2
- new net N$36: R19.1, U$165.P$1, U$165.P$2
- new net N$37: R20.1, U$168.P$1, U$168.P$2
- new net N$38: R17.1, U$169.P$1, U$169.P$2
- new net N$39: U$171.P1, U10.2
- new net N$40: R18.2, U$172.P$1, U$172.P$2, U9.EMITTER
- new net N$41: D6.3, R24.2
- new net N$42: D6.1, R23.2
- new net N$43: D6.2, R21.2
- new net N$44: R23.1, U$206.P$1, U$206.P$2
- new net N$45: R24.1, U$209.P$1, U$209.P$2
- new net N$46: R21.1, U$210.P$1, U$210.P$2
- new net N$47: U$212.P1, U12.2
- new net N$48: R22.2, U$213.P$1, U$213.P$2, U11.EMITTER
- new net N$9: D3.3, R12.2
Routing:
- net 3.3V4: track 0.00 -> 442.1 mm
- net 3.3V2: track 0.00 -> 442.1 mm
- net 3.3V5: track 0.00 -> 442.1 mm
- net 3.3V3: track 0.00 -> 442.1 mm
- net GND4: track 0.00 -> 281.8 mm, vias 0 -> 1
- net GND3: track 0.00 -> 281.8 mm, vias 0 -> 1
- net GND5: track 0.00 -> 281.8 mm, vias 0 -> 1
- net GND2: track 0.00 -> 281.8 mm, vias 0 -> 1
- net N$48: track 0.00 -> 30.8 mm, vias 0 -> 1
- net N$32: track 0.00 -> 30.8 mm, vias 0 -> 1
- net N$40: track 0.00 -> 30.8 mm, vias 0 -> 1
- net N$24: track 0.00 -> 30.8 mm, vias 0 -> 1
- net N$37: track 0.00 -> 23.0 mm
- net N$21: track 0.00 -> 23.0 mm
- net N$29: track 0.00 -> 23.0 mm
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Other:
- board size 111.5 x 119.6 mm -> 105.2 x 313.4 mm
- board text removed: "v-score"

Commit message: panel
Parts:
- U$112, U$153, U$194, U$235, U$34, U$71: device 003:TRI#COLOR_LED1 -> buzzard_labels (1):RGB_LED0
- U$130, U$171, U$212, U$23, U$47, U$89: value TAB_GATOR_MINI -> GATOR; device SparkFun-Connectors:TAB_GATOR_MINI -> SparkFun-Connectors:GATOR
- moved U$171 10.2 mm to (15.9, 231.9)
- moved U$212 10.2 mm to (15.9, 281.9)
- moved U$130 10.2 mm to (15.9, 181.9)
- moved U$23 10.2 mm to (15.9, 31.8)
- moved U$47 10.2 mm to (15.9, 81.8)
- moved U$89 10.2 mm to (15.9, 131.8)
- moved U$194 1.80 mm to (49.7, 231.8)
- moved U$235 1.80 mm to (49.7, 281.9)
- moved U$71 1.80 mm to (49.7, 81.7)
- moved U$34 1.80 mm to (49.7, 31.7)
- moved U$112 1.80 mm to (49.7, 131.8)
- moved U$153 1.80 mm to (49.7, 181.8)
Connections:
- net N$10: now also U$23.P$1, U$23.P$2; no longer U$23.P1
- net N$23: now also U$89.P$1, U$89.P$2; no longer U$89.P1
- net N$31: now also U$130.P$1, U$130.P$2; no longer U$130.P1
- net N$39: now also U$171.P$1, U$171.P$2; no longer U$171.P1
- net N$47: now also U$212.P$1, U$212.P$2; no longer U$212.P1
- net N$7: now also U$47.P$1, U$47.P$2; no longer U$47.P1
Routing:
- net N$7: track 15.0 -> 18.9 mm
- net N$23: track 15.0 -> 18.9 mm
- net N$10: track 15.0 -> 18.9 mm
- net N$39: track 15.0 -> 18.9 mm
- net N$31: track 15.0 -> 18.9 mm
- net N$47: track 15.0 -> 18.9 mm
